File: KiCad/ADCBreakout/ADCBreakout.sch (KiCad schematic (older format))
At the start: 2 parts, among them J1 CONN_01X08, U1 ADC122S101

Commit message: Added pinout/mapping for Rpi GPIO connector
Parts:
- U1: footprint Housings_SSOP:VSSOP-8_3.0x3.0mm_Pitch0.65mm -> BowlsEye:MyVSSOP-8_3.0x3.0mm_Pitch0.65mm
Changed lines of the file:
@@
 F 0 "U1" H 5325 2675 60  0000 C CNN
 F 1 "ADC122S101" H 5325 2225 60  0000 C CNN
-F 2 "Housings_SSOP:VSSOP-8_3.0x3.0mm_Pitch0.65mm" H 5325 2375 60  0001 C CNN
+F 2 "BowlsEye:MyVSSOP-8_3.0x3.0mm_Pitch0.65mm" H 5325 2375 60  0001 C CNN
 F 3 "" H 5325 2375 60  0001 C CNN
 	1    5325 2525
