File: KiCad/Shield/_autosave-Proto1.kicad_pcb (KiCad board)
At the start: 2 copper layers, 208.6 x 98.3 mm, 74 parts, among them J1 CONN_02X20, J10 CONN_01X02, J11 CONN_01X02, J2 CONN_01X04, J3 CONN_01X02, J4 CONN_01X02, J5 CONN_01X02, J6 CONN_01X02, J7 CONN_01X02, J8 CONN_01X02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

Commit message: added PCB and PDF of schematics
Parts:
- moved REF** 2.50 mm to (167.3, 49.7)
- moved REF** 2.50 mm to (167.3, 106.6)
Other:
- board text added: "Double check pin out for transistors! Double check dimensions/holes!"
- board text removed: "Double check pin out for transistors!"
Changed lines of the file:
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@@
   )
   (module Connectors:1pin (layer F.Cu)
-    (at 164.775 49.675)
+    (at 167.275 49.675)
     (descr "module 1 pin (ou trou mecanique de percage)")
     (tags DEV)
@@
   )
   (module Connectors:1pin (layer F.Cu)
-    (at 164.775 106.6)
+    (at 167.275 106.6)
     (descr "module 1 pin (ou trou mecanique de percage)")
     (tags DEV)
@@
     )
   )
-  (gr_text "Double check pin out for transistors!" (at 129.1 21.8) (layer Eco1.User)
+  (gr_text "Double check pin out for transistors!\nDouble check dimensions/holes!" (at 129.1 21.8) (layer Eco1.User)
     (effects (font (size 3 3) (thickness 0.3)))
   )
