File: KiCad/Shield/motorDriver.sch (KiCad schematic (older format))
At the start: 4 parts

Commit message: updated schematic
Connections:
- net GNDD: now also U?.1 (SenseA), U?.15 (SenseB)
- no-connect marks 2 -> 0
Changed lines of the file:
@@
 Text GLabel 5850 3000 2    35   Input ~ 0
 PHASE_B-
-NoConn ~ 5750 3500
-NoConn ~ 5750 3600
 $Comp
 L GNDD #PWR?
@@
 Wire Wire Line
 	4750 2800 4650 2800
+Wire Wire Line
+	5750 3500 5850 3500
+Wire Wire Line
+	5850 3500 5850 3700
+Wire Wire Line
+	5850 3600 5750 3600
+Connection ~ 5850 3600
+$Comp
+L GNDD #PWR?
+U 1 1 5AA879F1
+P 5850 3700
+F 0 "#PWR?" H 5850 3450 50  0001 C CNN
+F 1 "GNDD" H 5850 3575 50  0000 C CNN
+F 2 "" H 5850 3700 50  0001 C CNN
+F 3 "" H 5850 3700 50  0001 C CNN
+	1    5850 3700
+	1    0    0    -1
+$EndComp
 $EndSCHEMATC

Commit message: removed hello world
Parts:
- J2: renamed from J?; footprint (none) -> Sockets_MOLEX_KK-System:Socket_MOLEX-KK-RM2-54mm_Lock_4pin_straight
- U2: renamed from U?; footprint (none) -> TO_SOT_Packages_THT:TO-220-15_Vertical_StaggeredType1
- gave numbers to parts that had none: 2
Changed lines of the file:
@@
 $EndDescr
 $Comp
-L CONN_01X04 J?
+L CONN_01X04 J2
 U 1 1 5AA69EB0
 P 8375 2900
-F 0 "J?" H 8375 3150 50  0000 C CNN
+F 0 "J2" H 8375 3150 50  0000 C CNN
 F 1 "CONN_01X04" V 8475 2900 50  0000 C CNN
-F 2 "" H 8375 2900 50  0001 C CNN
+F 2 "Sockets_MOLEX_KK-System:Socket_MOLEX-KK-RM2-54mm_Lock_4pin_straight" H 8375 2900 50  0001 C CNN
 F 3 "" H 8375 2900 50  0001 C CNN
 	1    8375 2900
@@
 PHASE_B-
 $Comp
-L L298_TH U?
+L L298_TH U2
 U 1 1 5AA6A712
 P 5250 3250
-F 0 "U?" H 5250 3200 35  0000 C CNN
+F 0 "U2" H 5250 3200 35  0000 C CNN
 F 1 "L298_TH" H 5250 3300 35  0000 C CNN
-F 2 "" H 5250 3200 35  0001 C CNN
+F 2 "TO_SOT_Packages_THT:TO-220-15_Vertical_StaggeredType1" H 5250 3200 35  0001 C CNN
 F 3 "" H 5250 3200 35  0001 C CNN
 	1    5250 3250
@@
 PHASE_B-
 $Comp
-L GNDD #PWR?
+L GNDD #PWR012
 U 1 1 5AA6A83B
 P 4650 3900
-F 0 "#PWR?" H 4650 3650 50  0001 C CNN
+F 0 "#PWR012" H 4650 3650 50  0001 C CNN
 F 1 "GNDD" H 4650 3775 50  0000 C CNN
 F 2 "" H 4650 3900 50  0001 C CNN
@@
 MOTOR_2_2
 $Comp
-L C_Small C?
+L C_Small C2
 U 1 1 5AA6ACA6
 P 1000 1075
-F 0 "C?" H 1010 1145 50  0000 L CNN
+F 0 "C2" H 1010 1145 50  0000 L CNN
 F 1 "100nF" H 1010 995 50  0000 L CNN
 F 2 "" H 1000 1075 50  0001 C CNN
@@
 $EndComp
 $Comp
-L GNDD #PWR?
+L GNDD #PWR013
 U 1 1 5AA6AEAD
 P 1000 1225
-F 0 "#PWR?" H 1000 975 50  0001 C CNN
+F 0 "#PWR013" H 1000 975 50  0001 C CNN
 F 1 "GNDD" H 1000 1100 50  0000 C CNN
 F 2 "" H 1000 1225 50  0001 C CNN
@@
 MOTOR_VS
 $Comp
-L C_Small C?
+L C_Small C3
 U 1 1 5AA6B308
 P 1675 1075
-F 0 "C?" H 1685 1145 50  0000 L CNN
+F 0 "C3" H 1685 1145 50  0000 L CNN
 F 1 "100nF" H 1685 995 50  0000 L CNN
 F 2 "" H 1675 1075 50  0001 C CNN
@@
 $EndComp
 $Comp
-L GNDD #PWR?
+L GNDD #PWR014
 U 1 1 5AA6B30E
 P 1675 1225
-F 0 "#PWR?" H 1675 975 50  0001 C CNN
+F 0 "#PWR014" H 1675 975 50  0001 C CNN
 F 1 "GNDD" H 1675 1100 50  0000 C CNN
 F 2 "" H 1675 1225 50  0001 C CNN
@@
 Connection ~ 5850 3600
 $Comp
-L GNDD #PWR?
+L GNDD #PWR015
 U 1 1 5AA879F1
 P 5850 3700
-F 0 "#PWR?" H 5850 3450 50  0001 C CNN
+F 0 "#PWR015" H 5850 3450 50  0001 C CNN
 F 1 "GNDD" H 5850 3575 50  0000 C CNN
 F 2 "" H 5850 3700 50  0001 C CNN

Commit message: added PCB and PDF of schematics
Parts:
- C2, C3: footprint (none) -> Capacitors_THT:C_Rect_L7.2mm_W3.0mm_P5.00mm_FKS2_FKP2_MKS2_MKP2
- J2: footprint Sockets_MOLEX_KK-System:Socket_MOLEX-KK-RM2-54mm_Lock_4pin_straight -> Connectors_Terminal_Blocks:TerminalBlock_Altech_AK300-4_P5.00mm
Connections:
- net PHASE_A: now also J2.2 (P2); no longer J2.1 (P1)
- net PHASE_A-: now also J2.4 (P4); no longer J2.2 (P2)
- net PHASE_B-: now also J2.1 (P1); no longer J2.4 (P4)
Other:
- note removed: "double check power requirements"
Changed lines of the file:
@@
 LIBS:adc122s101
 LIBS:l298_th
+LIBS:transducer
 LIBS:Proto1-cache
 EELAYER 25 0
@@
 F 0 "J2" H 8375 3150 50  0000 C CNN
 F 1 "CONN_01X04" V 8475 2900 50  0000 C CNN
-F 2 "Sockets_MOLEX_KK-System:Socket_MOLEX-KK-RM2-54mm_Lock_4pin_straight" H 8375 2900 50  0001 C CNN
+F 2 "Connectors_Terminal_Blocks:TerminalBlock_Altech_AK300-4_P5.00mm" H 8375 2900 50  0001 C CNN
 F 3 "" H 8375 2900 50  0001 C CNN
 	1    8375 2900
 	1    0    0    -1
 $EndComp
-Text GLabel 8075 2750 0    35   Input ~ 0
+Text GLabel 8075 2850 0    35   Input ~ 0
 PHASE_A
-Text GLabel 8075 2850 0    35   Input ~ 0
+Text GLabel 8075 3050 0    35   Input ~ 0
 PHASE_A-
 Text GLabel 8075 2950 0    35   Input ~ 0
 PHASE_B
-Text GLabel 8075 3050 0    35   Input ~ 0
+Text GLabel 8075 2750 0    35   Input ~ 0
 PHASE_B-
 $Comp
@@
 PHASE_B-
 $Comp
-L GNDD #PWR012
+L GNDD #PWR016
 U 1 1 5AA6A83B
 P 4650 3900
-F 0 "#PWR012" H 4650 3650 50  0001 C CNN
+F 0 "#PWR016" H 4650 3650 50  0001 C CNN
 F 1 "GNDD" H 4650 3775 50  0000 C CNN
 F 2 "" H 4650 3900 50  0001 C CNN
@@
 F 0 "C2" H 1010 1145 50  0000 L CNN
 F 1 "100nF" H 1010 995 50  0000 L CNN
-F 2 "" H 1000 1075 50  0001 C CNN
+F 2 "Capacitors_THT:C_Rect_L7.2mm_W3.0mm_P5.00mm_FKS2_FKP2_MKS2_MKP2" H 1000 1075 50  0001 C CNN
 F 3 "" H 1000 1075 50  0001 C CNN
 	1    1000 1075
@@
 $EndComp
 $Comp
-L GNDD #PWR013
+L GNDD #PWR017
 U 1 1 5AA6AEAD
 P 1000 1225
-F 0 "#PWR013" H 1000 975 50  0001 C CNN
+F 0 "#PWR017" H 1000 975 50  0001 C CNN
 F 1 "GNDD" H 1000 1100 50  0000 C CNN
 F 2 "" H 1000 1225 50  0001 C CNN
@@
 	1    0    0    -1
 $EndComp
-Text Notes 4175 2500 0    35   ~ 0
-double check power requirements
 Text GLabel 1000 775  0    35   Input ~ 0
 +5V
@@
 F 0 "C3" H 1685 1145 50  0000 L CNN
 F 1 "100nF" H 1685 995 50  0000 L CNN
-F 2 "" H 1675 1075 50  0001 C CNN
+F 2 "Capacitors_THT:C_Rect_L7.2mm_W3.0mm_P5.00mm_FKS2_FKP2_MKS2_MKP2" H 1675 1075 50  0001 C CNN
 F 3 "" H 1675 1075 50  0001 C CNN
 	1    1675 1075
@@
 $EndComp
 $Comp
-L GNDD #PWR014
+L GNDD #PWR018
 U 1 1 5AA6B30E
 P 1675 1225
-F 0 "#PWR014" H 1675 975 50  0001 C CNN
+F 0 "#PWR018" H 1675 975 50  0001 C CNN
 F 1 "GNDD" H 1675 1100 50  0000 C CNN
 F 2 "" H 1675 1225 50  0001 C CNN
@@
 Connection ~ 5850 3600
 $Comp
-L GNDD #PWR015
+L GNDD #PWR019
 U 1 1 5AA879F1
 P 5850 3700
-F 0 "#PWR015" H 5850 3450 50  0001 C CNN
+F 0 "#PWR019" H 5850 3450 50  0001 C CNN
 F 1 "GNDD" H 5850 3575 50  0000 C CNN
 F 2 "" H 5850 3700 50  0001 C CNN
