File: KiCad/Shield/power.sch (KiCad schematic (older format))
At the start: 2 parts

Commit message: removed hello world
Parts:
- added C?: 10uF, symbol CP1_Small
- added C? (x2): 100nF, symbol C_Small
- added J?: CONN_01X02, symbol CONN_01X02
- added SW?: SW_SPDT, symbol SW_SPDT
- added U?: L7805, symbol L7805
- gave numbers to parts that had none: 2
Connections:
- net GNDREF: now also C?.2, C?.2, C?.2, J?.2 (P2), U?.2 (GND)
- new net: J?.1 (P1), SW?.2 (B)
- new net: C?.1, C?.1, SW?.3 (C), U?.1 (IN)
- new net +5V: C?.1, U?.3 (OUT)
- no-connect marks 0 -> 1
Changed lines of the file:
@@
 $EndDescr
 $Comp
-L GNDD #PWR?
+L GNDD #PWR01
 U 1 1 5AA6A86D
 P 1750 2200
-F 0 "#PWR?" H 1750 1950 50  0001 C CNN
+F 0 "#PWR01" H 1750 1950 50  0001 C CNN
 F 1 "GNDD" H 1750 2075 50  0000 C CNN
 F 2 "" H 1750 2200 50  0001 C CNN
@@
 $EndComp
 $Comp
-L GNDREF #PWR?
+L GNDREF #PWR02
 U 1 1 5AA6A887
 P 2150 2200
-F 0 "#PWR?" H 2150 1950 50  0001 C CNN
+F 0 "#PWR02" H 2150 1950 50  0001 C CNN
 F 1 "GNDREF" H 2150 2050 50  0000 C CNN
 F 2 "" H 2150 2200 50  0001 C CNN
@@
 $EndComp
 $Comp
-L GNDA #PWR?
+L GNDA #PWR03
 U 1 1 5AA6A8AD
 P 2550 2200
-F 0 "#PWR?" H 2550 1950 50  0001 C CNN
+F 0 "#PWR03" H 2550 1950 50  0001 C CNN
 F 1 "GNDA" H 2550 2050 50  0000 C CNN
 F 2 "" H 2550 2200 50  0001 C CNN
@@
 $EndComp
 $Comp
-L L_Small L?
+L L_Small L1
 U 1 1 5AA6A8CC
 P 1950 2150
-F 0 "L?" H 1980 2190 50  0000 L CNN
+F 0 "L1" H 1980 2190 50  0000 L CNN
 F 1 "100nH" H 1980 2110 50  0000 L CNN
 F 2 "" H 1950 2150 50  0001 C CNN
@@
 $EndComp
 $Comp
-L L_Small L?
+L L_Small L2
 U 1 1 5AA6A960
 P 2350 2150
-F 0 "L?" H 2380 2190 50  0000 L CNN
+F 0 "L2" H 2380 2190 50  0000 L CNN
 F 1 "100nH" H 2380 2110 50  0000 L CNN
 F 2 "" H 2350 2150 50  0001 C CNN
@@
 Text Notes 5125 3350 0    394  ~ 79
 TBC
+$Comp
+L SW_SPDT SW?
+U 1 1 5AAA7583
+P 2750 1100
+F 0 "SW?" H 2750 1270 50  0000 C CNN
+F 1 "SW_SPDT" H 2750 900 50  0000 C CNN
+F 2 "" H 2750 1100 50  0001 C CNN
+F 3 "" H 2750 1100 50  0001 C CNN
+	1    2750 1100
+	1    0    0    -1
+$EndComp
+Wire Wire Line
+	2050 1100 2550 1100
+NoConn ~ 2950 1000
+Wire Wire Line
+	2950 1200 3550 1200
+$Comp
+L CONN_01X02 J?
+U 1 1 5AAA7712
+P 1850 1150
+F 0 "J?" H 1850 1300 50  0000 C CNN
+F 1 "CONN_01X02" V 1950 1150 50  0000 C CNN
+F 2 "" H 1850 1150 50  0001 C CNN
+F 3 "" H 1850 1150 50  0001 C CNN
+	1    1850 1150
+	-1   0    0    -1
+$EndComp
+Wire Wire Line
+	2050 1200 2150 1200
+Wire Wire Line
+	2150 1200 2150 1250
+$Comp
+L GNDREF #PWR?
+U 1 1 5AAA78AF
+P 2150 1250
+F 0 "#PWR?" H 2150 1000 50  0001 C CNN
+F 1 "GNDREF" H 2150 1100 50  0000 C CNN
+F 2 "" H 2150 1250 50  0001 C CNN
+F 3 "" H 2150 1250 50  0001 C CNN
+	1    2150 1250
+	1    0    0    -1
+$EndComp
+$Comp
+L L7805 U?
+U 1 1 5AAA793B
+P 3850 1200
+F 0 "U?" H 3700 1325 50  0000 C CNN
+F 1 "L7805" H 3850 1325 50  0000 L CNN
+F 2 "" H 3875 1050 50  0001 L CIN
+F 3 "" H 3850 1150 50  0001 C CNN
+	1    3850 1200
+	1    0    0    -1
+$EndComp
+Wire Wire Line
+	3850 1500 3850 1600
+$Comp
+L GNDREF #PWR?
+U 1 1 5AAA7A31
+P 3850 1600
+F 0 "#PWR?" H 3850 1350 50  0001 C CNN
+F 1 "GNDREF" H 3850 1450 50  0000 C CNN
+F 2 "" H 3850 1600 50  0001 C CNN
+F 3 "" H 3850 1600 50  0001 C CNN
+	1    3850 1600
+	1    0    0    -1
+$EndComp
+Wire Wire Line
+	4150 1200 4375 1200
+Connection ~ 3350 1200
+Wire Wire Line
+	3350 1500 3350 1550
+Wire Wire Line
+	3350 1550 4250 1550
+Connection ~ 4250 1200
+Wire Wire Line
+	4250 1550 4250 1500
+Connection ~ 3850 1550
+Wire Wire Line
+	4250 1200 4250 1300
+Wire Wire Line
+	3350 1200 3350 1300
+Wire Wire Line
+	3075 1200 3075 1300
+Connection ~ 3075 1200
+$Comp
+L CP1_Small C?
+U 1 1 5AAA8061
+P 3075 1400
+F 0 "C?" H 3085 1470 50  0000 L CNN
+F 1 "10uF" H 3085 1320 50  0000 L CNN
+F 2 "" H 3075 1400 50  0001 C CNN
+F 3 "" H 3075 1400 50  0001 C CNN
+	1    3075 1400
+	1    0    0    -1
+$EndComp
+Wire Wire Line
+	3075 1500 3075 1600
+$Comp
+L GNDREF #PWR?
+U 1 1 5AAA80E0
+P 3075 1600
+F 0 "#PWR?" H 3075 1350 50  0001 C CNN
+F 1 "GNDREF" H 3075 1450 50  0000 C CNN
+F 2 "" H 3075 1600 50  0001 C CNN
+F 3 "" H 3075 1600 50  0001 C CNN
+	1    3075 1600
+	1    0    0    -1
+$EndComp
+$Comp
+L C_Small C?
+U 1 1 5AAA818F
+P 3350 1400
+F 0 "C?" H 3360 1470 50  0000 L CNN
+F 1 "100nF" H 3360 1320 50  0000 L CNN
+F 2 "" H 3350 1400 50  0001 C CNN
+F 3 "" H 3350 1400 50  0001 C CNN
+	1    3350 1400
+	1    0    0    -1
+$EndComp
+$Comp
+L C_Small C?
+U 1 1 5AAA8241
+P 4250 1400
+F 0 "C?" H 4260 1470 50  0000 L CNN
+F 1 "100nF" H 4260 1320 50  0000 L CNN
+F 2 "" H 4250 1400 50  0001 C CNN
+F 3 "" H 4250 1400 50  0001 C CNN
+	1    4250 1400
+	1    0    0    -1
+$EndComp
+Text GLabel 4375 1200 2    35   Input ~ 0
++5V
 $EndSCHEMATC

Commit message: added PCB and PDF of schematics
Parts:
- added C11, C22: 10uF, Capacitors_THT:CP_Radial_D5.0mm_P2.00mm, symbol CP1_Small
- added C20, C21: 100nF, Capacitors_THT:C_Rect_L7.2mm_W3.0mm_P5.00mm_FKS2_FKP2_MKS2_MKP2, symbol C_Small
- added D7: LED, LEDs:LED_D3.0mm, symbol LED
- added R19: R, Resistors_THT:R_Axial_DIN0207_L6.3mm_D2.5mm_P10.16mm_Horizontal, symbol R
- added U4: LD1117S33TR_SOT223, TO_SOT_Packages_THT:TO-220-3_Horizontal, symbol LD1117S33TR_SOT223
- C10, C9: renamed from C?; footprint (none) -> Capacitors_THT:C_Rect_L7.2mm_W3.0mm_P5.00mm_FKS2_FKP2_MKS2_MKP2
- C8: renamed from C?; footprint (none) -> Capacitors_THT:CP_Radial_D5.0mm_P2.00mm
- J7: renamed from J?; footprint (none) -> Connectors_Terminal_Blocks:TerminalBlock_Altech_AK300-2_P5.00mm
- L1: footprint (none) -> Inductors_THT:L_Axial_L24.0mm_D7.5mm_P7.62mm_Vertical_Fastron_MESC
- SW1: renamed from SW?; footprint (none) -> BowlsEye:SPDT
- U3: renamed from U?; value L7805 -> L78S05CV; footprint (none) -> TO_SOT_Packages_THT:TO-220-3_Horizontal
Connections:
- net +5V: now also C11.1, C20.1, U4.3 (VI)
- net GNDREF: now also C11.2, C20.2, C21.2, C22.2, R19.2, U4.1 (GND)
- net at C8.1, C9.1, SW1.3 (C)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: now also D7.2 (A)
- new net: D7.1 (K), R19.1
- new net +3V3: C21.1, C22.1, U4.2 (VO)
Other:
- note added: "max 2A output"
- note removed: "TBC"
- moved on the sheet: C10, C8, C9, SW1, U3
