File: KiCad/Shield/ultrasound.sch (KiCad schematic (older format))
At the start: 50 parts

Commit message: removed hello world
Parts:
- removed C? (x4): 100nF, symbol C_Small
- removed U? (x4): TL072, symbol TL072
- added U? (x4): LM324N, symbol LM324N
- gave numbers to parts that had none: 42
Connections:
- net +12V is gone; now on net +5V: C4.2, C5.2, C6.2, C7.2
- net +5V: now also U?.4 (V+), U?.4 (V+), U?.4 (V+), U?.4 (V+)
- net GNDD: now also U?.12 (+), U?.5 (+)
- net ULTRA_RX1_RAW: now also U?.3 (+)
- net ULTRA_RX2_RAW: now also U?.10 (+)
- net at C12.1, R5.1: now also U?.1
- net at R3.2, R5.2: now also U?.2 (-)
- net at C14.1, R7.1, R9.2: now also U?.6 (-)
- net at C14.2, C16.1, R9.1: now also U?.7
- net at C13.1, R6.1: now also U?.8
- net at R4.2, R6.2: now also U?.9 (-)
- net at C15.2, C17.1, R10.1: now also U?.14
- net at C15.1, R10.2, R8.1: now also U?.13 (-)

Commit message: added PCB and PDF of schematics
Parts:
- removed C5, C6, C7: 100nF, symbol C_Small
- removed D5, D6: D_Small, symbol D_Small
- added J10, J11, J8, J9: CONN_01X02, Connectors_Terminal_Blocks:TerminalBlock_Altech_AK300-2_P5.00mm, symbol CONN_01X02
- added U6, U7, U8, U9: transducer, BowlsEye:transducer, symbol transducer
- C12, C13, C14, C15, C16, C17, C18, C19, C4: footprint (none) -> Capacitors_THT:C_Rect_L7.2mm_W3.0mm_P5.00mm_FKS2_FKP2_MKS2_MKP2
- D1, D2, D3, D4: footprint (none) -> Diodes_THT:D_T-1_P10.16mm_Horizontal
- J3, J4, J5, J6: footprint (none) -> Connectors_Terminal_Blocks:TerminalBlock_Altech_AK300-2_P5.00mm
- R1, R10, R11, R12, R13, R14, R15, R16, R17, R18, R2, R3, R4, R5, R6, R7, R8, R9: footprint (none) -> Resistors_THT:R_Axial_DIN0207_L6.3mm_D2.5mm_P10.16mm_Horizontal
- U5: renamed from U?; footprint (none) -> Housings_DIP:DIP-14_W7.62mm_LongPads
- gave numbers to parts that had none: 1
Connections:
- net +5V: no longer J5.1 (P1), J6.1 (P1)
- net GNDD: now also U5.10 (+), U5.11 (V-), U5.11 (V-), U5.11 (V-), U5.11 (V-), J8.2 (P2), J9.2 (P2), U6.2 (-), U7.2 (-); no longer J5.2 (P2), J6.2 (P2), U5.5 (+)
- net ULTRA_RX1_RAW: now also J8.1 (P1), U6.1 (+)
- net ULTRA_RX2_RAW: now also U5.5 (+), J9.1 (P1), U7.1 (+); no longer U5.10 (+)
- net at Q1.3 (C): now also J5.2 (P2); no longer R17.1
- net at C14.1, R7.1, R9.2: now also U5.13 (-); no longer U5.6 (-)
- net at C14.2, C16.1, R9.1: now also U5.14; no longer U5.7
- net at C13.1, R6.1: now also U5.7; no longer U5.8
- net at R4.2, R6.2: now also U5.6 (-); no longer U5.9 (-)
- net at C15.1, R10.2, R8.1: now also U5.9 (-); no longer U5.13 (-)
- net at C15.2, C17.1, R10.1: now also U5.8; no longer U5.14
- net at Q2.3 (C): now also J6.2 (P2); no longer R18.1
- new net: J5.1 (P1), R17.1
- new net: J6.1 (P1), R18.1
- new net: J11.1 (P1), U9.1 (+)
- new net: J11.2 (P2), U9.2 (-)
- new net: J10.1 (P1), U8.1 (+)
- new net: J10.2 (P2), U8.2 (-)
Other:
- note removed: "ToDo:\nChange to Single Rail 5V Op Amps?"
- note removed: "to transducer"
- moved on the sheet: C12, C13, C14, C15, C16, C17, C18, C19, C4, D1, D2, D3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
