File: KiCad/Shield/Proto1.kicad_pcb (KiCad board)
At the start: 2 copper layers, 208.6 x 98.3 mm, 74 parts, among them J1 CONN_02X20, J10 CONN_01X02, J11 CONN_01X02, J2 CONN_01X04, J3 CONN_01X02, J4 CONN_01X02, J5 CONN_01X02, J6 CONN_01X02, J7 CONN_01X02, J8 CONN_01X02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

Commit message: updated PCB and added fab files/bom
Parts:
- removed L1: 100nH, Inductors_THT:L_Axial_L24.0mm_D7.5mm_P7.62mm_Vertical_Fastron_MESC
- added D5: LED, LEDs:LED_D3.0mm, F.Cu at (203.0, 64.7)
- added J14: GS2, Connectors:GS2, B.Cu at (94.7, 123.8)
- added J15: GS2, Connectors:GS2, B.Cu at (102.8, 81.8)
- added J17: GS2, Connectors:GS2, B.Cu at (102.7, 98.4)
- added J18: GS2, Connectors:GS2, B.Cu at (175.8, 64.7)
- added J19: GS2, Connectors:GS2, F.Cu at (98.5, 107.2)
- added J20: GS2, Connectors:GS2, B.Cu at (129.3, 105.8)
- added R21: R, Resistors_THT:R_Axial_DIN0207_L6.3mm_D2.5mm_P10.16mm_Horizontal, F.Cu at (199.8, 62.0)
- added REF**: 1pin, Connectors:1pin, F.Cu at (37.0, 79.5)
- added REF**: 1pin, Connectors:1pin, F.Cu at (37.0, 45.0)
- moved J11 29.3 mm to (49.5, 95.5), turned to 180 degrees
- moved J9 29.1 mm to (29.5, 95.5), turned to 180 degrees
- moved J8 25.6 mm to (29.5, 61.0), turned to 180 degrees
- moved J10 25.1 mm to (49.5, 61.0), turned to 180 degrees
- moved U9 12.5 mm to (47.0, 86.5), turned to 180 degrees
- moved U7 12.5 mm to (27.0, 86.5), turned to 180 degrees
- moved U8 8.86 mm to (47.0, 52.0), turned to 180 degrees
- moved U6 8.86 mm to (27.0, 52.0), turned to 180 degrees
- moved REF** 4.10 mm to (212.8, 108.8)
- moved C14 3.83 mm to (134.7, 78.6)
- moved C15 3.83 mm to (134.7, 82.6)
- moved C16 3.83 mm to (147.9, 74.8)
- moved C19 3.83 mm to (159.7, 87.3)
- moved C22 3.83 mm to (121.1, 105.8)
- moved C4 3.83 mm to (112.5, 79.8)
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Connections:
- net Net-(C8-Pad1) renamed +Vs
- C10 pad 2: GNDREF -> GNDD
- C11 pad 2: GNDREF -> GNDD
- C20 pad 2: GNDREF -> GNDD
- C21 pad 2: GNDREF -> GNDD
- C22 pad 2: GNDREF -> GNDD
- C8 pad 2: GNDREF -> GNDD
- C9 pad 2: GNDREF -> GNDD
- J1 pad 1: +3V3 -> Net-(J1-Pad1)
- J1 pad 7: Net-(J1-Pad7) -> DEBUG_PIN
- J7 pad 2: GNDREF -> GNDD
- R19 pad 2: GNDREF -> GNDD
- U3 pad 2: GNDREF -> GNDD
- U4 pad 1: GNDREF -> GNDD
Routing:
- net GNDD: track 8.91 -> 62.1 mm, vias 3 -> 8
- net Net-(J11-Pad2): track 0.00 -> 16.3 mm, vias 0 -> 1
- net Net-(J10-Pad2): track 0.00 -> 16.3 mm, vias 0 -> 1
- net Net-(J11-Pad1): track 0.00 -> 15.6 mm, vias 0 -> 1
- net Net-(J10-Pad1): track 0.00 -> 15.6 mm, vias 0 -> 1
- net ULTRA_RX2_RAW: track 38.9 -> 54.5 mm, vias 1 -> 2
- net ULTRA_RX1_RAW: track 38.5 -> 54.2 mm, vias 0 -> 1
- net DEBUG_PIN: track 0.00 -> 6.63 mm
- net Net-(D5-Pad1): track 0.00 -> 4.29 mm
- net +5V: track 253.4 -> 257.1 mm, vias 2 -> 3
- net +3V3: track 121.0 -> 118.2 mm
- net MOTOR_ENA: track 52.8 -> 54.4 mm
- net +Vs: track 32.8 -> 31.5 mm
- net PHASE_B: track 109.3 -> 110.1 mm
- net PHASE_A: track 95.1 -> 95.8 mm
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- added copper zone on F.Cu, net GNDD
- removed copper zone on B.Cu, net GNDREF
- removed copper zone on F.Cu, net GNDREF
Other:
- board size 208.6 x 98.3 mm -> 204.1 x 93.3 mm
- board text added: "BOTTOM ASSEMBLY"
- board text added: "BowlsEye 2018"
- board text added: "RX"
- board text added: "TOP ASSEMBLY"
- board text added: "TX"
- board text removed: "BowlsEye Layout by H Leicester 2018"
- board text removed: "Double check pin out for transistors!"
- board text removed: "ToDo: Add mounting holes for transducer boards"
