File: KiCad/Shield/rPi.sch (KiCad schematic (older format))
At the start: 3 parts

Commit message: updated schematic
Connections:
- net MOTOR_1_1: now reaches J?.11 (P11)
- net MOTOR_1_2: now reaches J?.13 (P13)
- net MOTOR_1_3: now reaches J?.15 (P15)
- net MOTOR_1_4: now reaches J?.16 (P16)
- net MOTOR_ENA: now reaches J?.3 (P3)
- net MOTOR_ENB: now reaches J?.5 (P5)
Other:
- note added: "ToDo:\nAdd ref/reg supply for ADC"
- note removed: "ToDo:\nAdd motor driver EnA, EnB\nAdd motor driver Control signals\nAdd ref/reg supply for ADC"
Changed lines of the file:
@@
 $EndComp
 Wire Wire Line
-	4850 3425 4450 3425
+	4250 3425 4850 3425
 $Comp
 L GNDD #PWR?
 U 1 1 5AA7FC0B
-P 4450 3475
-F 0 "#PWR?" H 4450 3225 50  0001 C CNN
-F 1 "GNDD" H 4450 3350 50  0000 C CNN
-F 2 "" H 4450 3475 50  0001 C CNN
-F 3 "" H 4450 3475 50  0001 C CNN
-	1    4450 3475
+P 4250 3475
+F 0 "#PWR?" H 4250 3225 50  0001 C CNN
+F 1 "GNDD" H 4250 3350 50  0000 C CNN
+F 2 "" H 4250 3475 50  0001 C CNN
+F 3 "" H 4250 3475 50  0001 C CNN
+	1    4250 3475
 	1    0    0    -1
 $EndComp
@@
 	5350 4425 5950 4425
 Wire Wire Line
-	5350 4625 5950 4625
-Wire Wire Line
 	4850 4925 4750 4925
 Wire Wire Line
 	4750 4925 4750 4975
-Wire Wire Line
-	5950 4625 5950 4675
 Wire Wire Line
 	5950 4425 5950 4475
@@
 Wire Wire Line
 	5950 3225 5950 3275
-Wire Wire Line
-	4450 3425 4450 3475
 Wire Wire Line
 	4650 4225 4650 4275
@@
 L GNDD #PWR?
 U 1 1 5AA7FEE1
-P 5950 4675
-F 0 "#PWR?" H 5950 4425 50  0001 C CNN
-F 1 "GNDD" H 5950 4550 50  0000 C CNN
-F 2 "" H 5950 4675 50  0001 C CNN
-F 3 "" H 5950 4675 50  0001 C CNN
-	1    5950 4675
+P 5550 4675
+F 0 "#PWR?" H 5550 4425 50  0001 C CNN
+F 1 "GNDD" H 5550 4550 50  0000 C CNN
+F 2 "" H 5550 4675 50  0001 C CNN
+F 3 "" H 5550 4675 50  0001 C CNN
+	1    5550 4675
 	1    0    0    -1
 $EndComp
@@
 	5450 4525 5350 4525
 Text Notes 1300 7050 0    197  ~ 39
-ToDo:\nAdd motor driver EnA, EnB\nAdd motor driver Control signals\nAdd ref/reg supply for ADC
-Wire Notes Line
-	1150 5600 6350 5600
-Wire Notes Line
-	1150 5600 1150 7225
-Wire Notes Line
-	1150 7225 6350 7225
-Wire Notes Line
-	6350 7225 6350 5600
+ToDo:\nAdd ref/reg supply for ADC
 Wire Wire Line
 	7425 3975 7425 4075
@@
 	7600 4325 7425 4325
 Connection ~ 7425 4325
+Wire Wire Line
+	4850 3525 4750 3525
+Wire Wire Line
+	4850 3625 4750 3625
+Wire Wire Line
+	4850 3725 4750 3725
+Wire Wire Line
+	5350 3725 5450 3725
+Text GLabel 4750 3525 0    35   Input ~ 0
+MOTOR_1_1
+Text GLabel 4750 3625 0    35   Input ~ 0
+MOTOR_1_2
+Text GLabel 4750 3725 0    35   Input ~ 0
+MOTOR_1_3
+Text GLabel 5450 3725 2    35   Input ~ 0
+MOTOR_1_4
+Wire Wire Line
+	4850 3125 4750 3125
+Text GLabel 4750 3125 0    35   Input ~ 0
+MOTOR_ENA
+Text GLabel 4750 3225 0    35   Input ~ 0
+MOTOR_ENB
+Wire Notes Line
+	1150 7225 1150 6325
+Wire Notes Line
+	1150 6325 5550 6325
+Wire Notes Line
+	5550 6325 5550 7225
+Wire Notes Line
+	5550 7225 1150 7225
+Wire Wire Line
+	4750 3225 4850 3225
+Wire Wire Line
+	4250 3425 4250 3475
+Wire Wire Line
+	5350 4625 5550 4625
+Wire Wire Line
+	5550 4625 5550 4675
 $EndSCHEMATC

Commit message: removed hello world
Parts:
- J1: renamed from J?; footprint (none) -> Pin_Headers:Pin_Header_Straight_2x20_Pitch2.54mm
- U1: renamed from U?; footprint (none) -> BowlsEye:MyVSSOP-8_3.0x3.0mm_Pitch0.65mm
- gave numbers to parts that had none: 1
Connections:
- net MOTOR_1_3 renamed MOTOR_2_1
- net MOTOR_1_4 renamed MOTOR_2_2
Changed lines of the file:
@@
 $EndDescr
 $Comp
-L CONN_02X20 J?
+L CONN_02X20 J1
 U 1 1 5AA699F4
 P 5100 3975
-F 0 "J?" H 5100 5025 50  0000 C CNN
+F 0 "J1" H 5100 5025 50  0000 C CNN
 F 1 "CONN_02X20" V 5100 3975 50  0000 C CNN
-F 2 "" H 5100 3025 50  0001 C CNN
+F 2 "Pin_Headers:Pin_Header_Straight_2x20_Pitch2.54mm" H 5100 3025 50  0001 C CNN
 F 3 "" H 5100 3025 50  0001 C CNN
 	1    5100 3975
@@
 	4650 4225 4850 4225
 $Comp
-L GNDD #PWR?
+L GNDD #PWR04
 U 1 1 5AA69E6F
 P 4650 4275
-F 0 "#PWR?" H 4650 4025 50  0001 C CNN
+F 0 "#PWR04" H 4650 4025 50  0001 C CNN
 F 1 "GNDD" H 4650 4150 50  0000 C CNN
 F 2 "" H 4650 4275 50  0001 C CNN
@@
 $EndComp
 $Comp
-L ADC122S101 U?
+L ADC122S101 U1
 U 1 1 5AA799C1
 P 8575 4075
-F 0 "U?" H 8575 4225 60  0000 C CNN
+F 0 "U1" H 8575 4225 60  0000 C CNN
 F 1 "ADC122S101" H 8575 3775 60  0000 C CNN
-F 2 "" H 8575 3925 60  0001 C CNN
+F 2 "BowlsEye:MyVSSOP-8_3.0x3.0mm_Pitch0.65mm" H 8575 3925 60  0001 C CNN
 F 3 "" H 8575 3925 60  0001 C CNN
 	1    8575 4075
@@
 Wire Wire Line
 	9025 4025 9125 4025
-Text GLabel 9125 4025 2    35   Input ~ 0
-SPI_MISO
 Wire Wire Line
 	9025 4125 9125 4125
-Text GLabel 9125 4125 2    35   Input ~ 0
-SPI_MOSI
 Wire Wire Line
 	9025 3925 9125 3925
@@
 	5350 3925 5950 3925
 $Comp
-L GNDD #PWR?
+L GNDD #PWR05
 U 1 1 5AA7FB9C
 P 5950 3975
-F 0 "#PWR?" H 5950 3725 50  0001 C CNN
+F 0 "#PWR05" H 5950 3725 50  0001 C CNN
 F 1 "GNDD" H 5950 3850 50  0000 C CNN
 F 2 "" H 5950 3975 50  0001 C CNN
@@
 	4250 3425 4850 3425
 $Comp
-L GNDD #PWR?
+L GNDD #PWR06
 U 1 1 5AA7FC0B
 P 4250 3475
-F 0 "#PWR?" H 4250 3225 50  0001 C CNN
+F 0 "#PWR06" H 4250 3225 50  0001 C CNN
 F 1 "GNDD" H 4250 3350 50  0000 C CNN
 F 2 "" H 4250 3475 50  0001 C CNN
@@
 	5350 3225 5950 3225
 $Comp
-L GNDD #PWR?
+L GNDD #PWR07
 U 1 1 5AA7FC6C
 P 5950 3275
-F 0 "#PWR?" H 5950 3025 50  0001 C CNN
+F 0 "#PWR07" H 5950 3025 50  0001 C CNN
 F 1 "GNDD" H 5950 3150 50  0000 C CNN
 F 2 "" H 5950 3275 50  0001 C CNN
@@
 	4650 4225 4650 4275
 $Comp
-L GNDD #PWR?
+L GNDD #PWR08
 U 1 1 5AA7FED0
 P 4750 4975
-F 0 "#PWR?" H 4750 4725 50  0001 C CNN
+F 0 "#PWR08" H 4750 4725 50  0001 C CNN
 F 1 "GNDD" H 4750 4850 50  0000 C CNN
 F 2 "" H 4750 4975 50  0001 C CNN
@@
 $EndComp
 $Comp
-L GNDD #PWR?
+L GNDD #PWR09
 U 1 1 5AA7FEE1
 P 5550 4675
-F 0 "#PWR?" H 5550 4425 50  0001 C CNN
+F 0 "#PWR09" H 5550 4425 50  0001 C CNN
 F 1 "GNDD" H 5550 4550 50  0000 C CNN
 F 2 "" H 5550 4675 50  0001 C CNN
@@
 $EndComp
 $Comp
-L GNDD #PWR?
+L GNDD #PWR010
 U 1 1 5AA7FEF2
 P 5950 4475
-F 0 "#PWR?" H 5950 4225 50  0001 C CNN
+F 0 "#PWR010" H 5950 4225 50  0001 C CNN
 F 1 "GNDD" H 5950 4350 50  0000 C CNN
 F 2 "" H 5950 4475 50  0001 C CNN
@@
 	7425 3975 7425 4075
 $Comp
-L C_Small C?
+L C_Small C1
 U 1 1 5AA8045B
 P 7425 4175
-F 0 "C?" H 7435 4245 50  0000 L CNN
+F 0 "C1" H 7435 4245 50  0000 L CNN
 F 1 "100nF" H 7435 4095 50  0000 L CNN
 F 2 "" H 7425 4175 50  0001 C CNN
@@
 Connection ~ 7425 4025
 $Comp
-L GNDD #PWR?
+L GNDD #PWR011
 U 1 1 5AA804FE
 P 7425 4375
-F 0 "#PWR?" H 7425 4125 50  0001 C CNN
+F 0 "#PWR011" H 7425 4125 50  0001 C CNN
 F 1 "GNDD" H 7425 4250 50  0000 C CNN
 F 2 "" H 7425 4375 50  0001 C CNN
@@
 MOTOR_1_2
 Text GLabel 4750 3725 0    35   Input ~ 0
-MOTOR_1_3
+MOTOR_2_1
 Text GLabel 5450 3725 2    35   Input ~ 0
-MOTOR_1_4
+MOTOR_2_2
 Wire Wire Line
 	4850 3125 4750 3125
@@
 Wire Wire Line
 	5550 4625 5550 4675
+Text GLabel 9125 4025 2    35   Input ~ 0
+SPI_MISO
+Text GLabel 9125 4125 2    35   Input ~ 0
+SPI_MOSI
 $EndSCHEMATC

Commit message: added PCB and PDF of schematics
Parts:
- added R20: 0R, Resistors_THT:R_Axial_DIN0207_L6.3mm_D2.5mm_P10.16mm_Horizontal, symbol R
- C1: footprint (none) -> Capacitors_THT:C_Rect_L7.2mm_W3.0mm_P5.00mm_FKS2_FKP2_MKS2_MKP2
Connections:
- net MOTOR_1_1: now also J1.15 (P15); no longer J1.11 (P11)
- net MOTOR_2_1: now also J1.5 (P5); no longer J1.15 (P15)
- net MOTOR_2_2: now also J1.3 (P3); no longer J1.16 (P16)
- net MOTOR_ENA: now also J1.8 (P8); no longer J1.3 (P3)
- net MOTOR_ENB: now also J1.11 (P11); no longer J1.5 (P5)
- net SPI_NSS0: now also R20.1, R20.2
- net ULTRA_RX1: now also U1.4 (IN2); no longer U1.5 (IN1)
- net ULTRA_RX2: now also U1.5 (IN1); no longer U1.4 (IN2)
- net ULTRA_TX1: now also J1.32 (P32); no longer J1.33 (P33)
- net ULTRA_TX2: now also J1.33 (P33); no longer J1.32 (P32)
- no-connect marks 0 -> 19
Other:
- note removed: "ToDo:\nAdd ref/reg supply for ADC"

Commit message: updated PCB and added fab files/bom
Parts:
- added D5: LED, LEDs:LED_D3.0mm, symbol LED
- added R21: R, Resistors_THT:R_Axial_DIN0207_L6.3mm_D2.5mm_P10.16mm_Horizontal, symbol R
- C1, J1, R20: part# (none) -> UofG
- U1: part# (none) -> ADC122S101CIMM/NOPB; rs# (none) -> 651-2278
Connections:
- net +3V3: no longer J1.1 (P1)
- net GNDD: now also R21.2
- net DEBUG_PIN: now reaches J1.7 (P7)
- net DEBUG_PIN: now also D5.2 (A)
- new net: D5.1 (K), R21.1
