File: KiCad/Shield/Proto2/power.sch (KiCad schematic (older format))
At the start: 19 parts, among them J14 GS2, J15 GS2, J17 GS2, J18 GS2, J19 GS2, J20 GS2, J7 CONN_01X02, SW1 SW_SPDT, U3 L78S05CV, U4 LD1117S33TR_SOT223

Commit message: Finished proto2 board
Parts:
- removed J7: CONN_01X02, Connectors_Terminal_Blocks:TerminalBlock_Altech_AK300-2_P5.00mm, symbol CONN_01X02
- added J7: CONN_01X04, Connectors_Molex:Molex_KK-41791-04_04x3.96mm_Straight, symbol CONN_01X04
Connections:
- net GNDD: now also J7.4 (P4)
- net at SW1.2 (B): now also J7.1 (P1)
- no-connect marks 1 -> 3
Changed lines of the file:
@@
 LIBS:l298_th
 LIBS:transducer
+LIBS:Proto2-cache
 EELAYER 25 0
 EELAYER END
@@
 $EndComp
 $Comp
-L CONN_01X02 J7
-U 1 1 5AAA7712
-P 1850 1150
-F 0 "J7" H 1850 1300 50  0000 C CNN
-F 1 "CONN_01X02" V 1950 1150 50  0000 C CNN
-F 2 "Connectors_Terminal_Blocks:TerminalBlock_Altech_AK300-2_P5.00mm" H 1850 1150 50  0001 C CNN
-F 3 "" H 1850 1150 50  0001 C CNN
-F 4 "UofG" H 1850 1400 50  0001 C CNN "part#"
-	1    1850 1150
-	-1   0    0    -1
-$EndComp
-$Comp
 L CP1_Small C8
 U 1 1 5AAA8061
@@
 $EndComp
 $Comp
-L GNDD #PWR01
+L GNDD #PWR1
 U 1 1 5AABC881
-P 2150 1250
-F 0 "#PWR01" H 2150 1000 50  0001 C CNN
-F 1 "GNDD" H 2150 1125 50  0000 C CNN
-F 2 "" H 2150 1250 50  0001 C CNN
-F 3 "" H 2150 1250 50  0001 C CNN
-	1    2150 1250
-	1    0    0    -1
-$EndComp
-$Comp
-L GNDD #PWR02
+P 2150 1450
+F 0 "#PWR1" H 2150 1200 50  0001 C CNN
+F 1 "GNDD" H 2150 1325 50  0000 C CNN
+F 2 "" H 2150 1450 50  0001 C CNN
+F 3 "" H 2150 1450 50  0001 C CNN
+	1    2150 1450
+	1    0    0    -1
+$EndComp
+$Comp
+L GNDD #PWR2
 U 1 1 5AABC94B
 P 3150 2000
-F 0 "#PWR02" H 3150 1750 50  0001 C CNN
+F 0 "#PWR2" H 3150 1750 50  0001 C CNN
 F 1 "GNDD" H 3150 1875 50  0000 C CNN
 F 2 "" H 3150 2000 50  0001 C CNN
@@
 $EndComp
 $Comp
-L GNDD #PWR03
+L GNDD #PWR3
 U 1 1 5AABC9A2
 P 4150 1600
-F 0 "#PWR03" H 4150 1350 50  0001 C CNN
+F 0 "#PWR3" H 4150 1350 50  0001 C CNN
 F 1 "GNDD" H 4150 1475 50  0000 C CNN
 F 2 "" H 4150 1600 50  0001 C CNN
@@
 	3050 1200 3850 1200
 Wire Wire Line
-	2050 1200 2150 1200
-Wire Wire Line
-	2150 1200 2150 1250
+	2050 1400 2150 1400
+Wire Wire Line
+	2150 1400 2150 1450
 Wire Wire Line
 	4150 1500 4150 1600
@@
 NoConn ~ 2650 1000
 $Comp
-L GNDD #PWR04
+L GNDD #PWR4
 U 1 1 5AABCA3D
 P 5975 1600
-F 0 "#PWR04" H 5975 1350 50  0001 C CNN
+F 0 "#PWR4" H 5975 1350 50  0001 C CNN
 F 1 "GNDD" H 5975 1475 50  0000 C CNN
 F 2 "" H 5975 1600 50  0001 C CNN
@@
 	1    0    0    -1
 $EndComp
+$Comp
+L CONN_01X04 J7
+U 1 1 5ACC34AE
+P 1850 1250
+F 0 "J7" H 1850 1500 50  0000 C CNN
+F 1 "CONN_01X04" V 1950 1250 50  0000 C CNN
+F 2 "Connectors_Molex:Molex_KK-41791-04_04x3.96mm_Straight" H 1850 1250 50  0001 C CNN
+F 3 "" H 1850 1250 50  0001 C CNN
+	1    1850 1250
+	-1   0    0    -1
+$EndComp
+NoConn ~ 2050 1200
+NoConn ~ 2050 1300
 $EndSCHEMATC
